File: TinyLamp.kicad_pcb (KiCad board)
At the start: 2 copper layers, 350 x 12 mm, 2 parts, among them J1 Conn_Coaxial_Small, U1 CH592F

Commit message: First commit
Parts:
- added C1: 0.1uF, Capacitor_SMD:C_0402_1005Metric, F.Cu at (97.0, 60.5)
- added C2: 0.1uF, Capacitor_SMD:C_0402_1005Metric, F.Cu at (96.0, 52.0)
- added C3: 0.1uF, Capacitor_SMD:C_0402_1005Metric, F.Cu at (92.0, 44.5)
- added C4: 0.1uF, Capacitor_SMD:C_0402_1005Metric, F.Cu at (92.5, 55.0)
- added C5: 1uF, Capacitor_SMD:C_0402_1005Metric, F.Cu at (90.5, 52.0)
- added L1: 22uH, Inductor_SMD:L_0402_1005Metric, F.Cu at (93.5, 52.0)
- added U2: XC6206P332MR, Package_TO_SOT_SMD:SOT-23-3, F.Cu at (96.5, 56.0)
- added Y1: 32M, Crystal:Crystal_SMD_3225-4Pin_3.2x2.5mm, F.Cu at (95.0, 42.5)
- J1: moved to B.Cu
- moved U1 67.3 mm to (95.2, 47.5), turned to 90 degrees
- moved J1 59.0 mm to (90.0, 38.0), turned to 180 degrees
Connections:
- J1 pad 1: unconnected-(J1-In-Pad1) -> Net-(J1-In)
- J1 pad 2: unconnected-(J1-Ext-Pad2) -> GND
- U1 pad 18: unconnected-(U1-~{X32MO}-Pad18) -> Net-(U1-~{X32MO})
- U1 pad 19: unconnected-(U1-X32MI-Pad19) -> Net-(U1-X32MI)
- U1 pad 20: unconnected-(U1-VINTA-Pad20) -> VCC
- U1 pad 21: unconnected-(U1-ANT-Pad21) -> Net-(J1-In)
- U1 pad 22: unconnected-(U1-VDCIA-Pad22) -> Net-(U1-VDCIA)
- U1 pad 29: unconnected-(U1-GND-Pad29) -> GND
- U1 pad 3: unconnected-(U1-VDCID-Pad3) -> Net-(U1-VDCIA)
- U1 pad 4: unconnected-(U1-VSW-Pad4) -> Net-(U1-VSW)
- U1 pad 5: GND -> VCC
Routing:
- net GND: track 0.00 -> 8.91 mm
- net VCC: track 0.00 -> 8.34 mm
- net Net-(U1-VDCIA): track 0.00 -> 8.32 mm
- net Net-(J1-In): track 0.00 -> 8.09 mm, vias 0 -> 1
- net +5V: track 0.00 -> 3.39 mm
- net Net-(U1-VSW): track 0.00 -> 3.03 mm
- net Net-(U1-~{X32MO}): track 0.00 -> 2.89 mm
- net Net-(U1-X32MI): track 0.00 -> 2.87 mm
Other:
- board size 350 x 12 mm -> 12 x 350 mm

Commit message: Core
Parts:
- added Y2: 32.768K, Crystal:Crystal_SMD_1210-4Pin_1.2x1.0mm, F.Cu at (92.0, 50.5)
- C3: value 0.1uF -> 0.47uF
- J1: moved to F.Cu
- moved C3 0.48 mm to (92.0, 44.0), turned to 90 degrees
- turned J1 to 0 degrees
Connections:
- C3 pad 1: VCC -> Net-(U1-VINTA)
- U1 pad 1: /X32KI -> Net-(U1-PA11)
- U1 pad 2: /X32KO -> Net-(U1-PA10)
- U1 pad 20: VCC -> Net-(U1-VINTA)
Routing:
- net VCC: track 8.34 -> 5.03 mm
- net Net-(U1-VINTA): track 0.00 -> 2.98 mm
- net Net-(U1-PA10): track 0.00 -> 2.83 mm
- net Net-(U1-PA11): track 0.00 -> 1.86 mm
- net Net-(J1-In): track 8.09 -> 9.39 mm, vias 1 -> 0

Commit message: Core
Parts:
- added U3: Opamp_Dual, Package_SO:VSSOP-8_2.3x2mm_P0.5mm, B.Cu at (91.4, 60.7)
Routing:
- net Net-(U1-VDCIA): track 8.32 -> 15.5 mm
- net VCC: track 5.03 -> 6.10 mm, vias 0 -> 1
- net unconnected-(U1-PA8-Pad6): track 0.00 -> 0.98 mm, vias 0 -> 1
- net unconnected-(U1-PA9-Pad7): track 0.00 -> 0.47 mm, vias 0 -> 1

Commit message: Core
Parts:
- moved U3 2.84 mm to (91.0, 63.5)
Routing:
- net VCC: track 6.10 -> 15.5 mm
- net GND: track 8.91 -> 12.2 mm, vias 0 -> 4
Changed lines of the file:
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@@
 	(footprint "Package_SO:VSSOP-8_2.3x2mm_P0.5mm"
 		(layer "B.Cu")
-		(at 91.44 60.695 90)
+		(at 91 63.5 90)
 		(descr "VSSOP, 8 Pin (https://www.jedec.org/standards-documents/docs/mo-187-f)")
 		(tags "VSSOP SO JEDEC-MO-187-CA Texas_DCU0008A")
@@
 	)
 	(segment
+		(start 95 47.5)
+		(end 94.5 48)
+		(width 0.2)
+		(layer "F.Cu")
+		(net "GND")
+	)
+	(segment
 		(start 96.48 52)
 		(end 96.48 53.9425)
@@
 	)
 	(segment
+		(start 95 47.5)
+		(end 94.5 47)
+		(width 0.2)
+		(layer "F.Cu")
+		(net "GND")
+	)
+	(segment
+		(start 95.5 47.5)
+		(end 96 48)
+		(width 0.2)
+		(layer "F.Cu")
+		(net "GND")
+	)
+	(segment
 		(start 97.4 54.8625)
 		(end 97.4 55.4)
@@
 	)
 	(segment
+		(start 95.175 47.5)
+		(end 95 47.5)
+		(width 0.2)
+		(layer "F.Cu")
+		(net "GND")
+	)
+	(segment
+		(start 95.5 47.5)
+		(end 96 47)
+		(width 0.2)
+		(layer "F.Cu")
+		(net "GND")
+	)
+	(segment
 		(start 97.48 55.48)
 		(end 97.48 60.5)
 		(width 0.2)
 		(layer "F.Cu")
+		(net "GND")
+	)
+	(segment
+		(start 95.175 47.5)
+		(end 95.5 47.5)
+		(width 0.2)
+		(layer "F.Cu")
+		(net "GND")
+	)
+	(via
+		(at 96 47)
+		(size 0.6)
+		(drill 0.3)
+		(layers "F.Cu" "B.Cu")
+		(net "GND")
+	)
+	(via
+		(at 94.5 47)
+		(size 0.6)
+		(drill 0.3)
+		(layers "F.Cu" "B.Cu")
+		(net "GND")
+	)
+	(via
+		(at 94.5 48)
+		(size 0.6)
+		(drill 0.3)
+		(layers "F.Cu" "B.Cu")
+		(net "GND")
+	)
+	(via
+		(at 96 48)
+		(size 0.6)
+		(drill 0.3)
+		(layers "F.Cu" "B.Cu")
 		(net "GND")
 	)
@@
 		(net "VCC")
 	)
+	(segment
+		(start 91.75 62.1)
+		(end 91.75 57.25)
+		(width 0.2)
+		(layer "B.Cu")
+		(net "VCC")
+	)
+	(segment
+		(start 91.75 57.25)
+		(end 95 54)
+		(width 0.2)
+		(layer "B.Cu")
+		(net "VCC")
+	)

Commit message: Touch
Parts:
- removed U3: Opamp_Dual, Package_SO:VSSOP-8_2.3x2mm_P0.5mm
Connections:
- U1 pad 6: unconnected-(U1-PA8-Pad6) -> /TCH0
- U1 pad 7: unconnected-(U1-PA9-Pad7) -> /TCH1
Routing:
- net /TCH1: track 0.00 -> 13.7 mm, vias 0 -> 1
- net VCC: track 15.5 -> 6.10 mm
- net unconnected-(U1-PA8-Pad6): track 0.98 -> 0.00 mm, vias 1 -> 0
- net /TCH0: track 0.00 -> 0.98 mm, vias 0 -> 1
- net unconnected-(U1-PA9-Pad7): track 0.47 -> 0.00 mm, vias 1 -> 0
- net (no net): vias 0 -> 3
- added copper zone on B.Cu, net /TCH0
- added copper zone on B.Cu, net /TCH1
