File: TinyLamp.kicad_sch (KiCad schematic)
At the start: 0 parts

Commit message: First commit
Parts:
- added J1: Conn_Coaxial_Small, Connector_Coaxial:U.FL_Molex_MCRF_73412-0110_Vertical, symbol Connector:Conn_Coaxial_Small
- added U1: CH592F, Package_DFN_QFN:WQFN-28-1EP_4x4mm_P0.4mm_EP2.7x2.7mm, symbol MCU_WCH_RiscV:CH592F
Connections:
- new net GND: U1.5 (VDD33/VIO33)
- new net X32KI: U1.1 (PA11)
- new net X32KO: U1.2 (PA10)

Commit message: First commit
Parts:
- added C1, C2, C3, C4: 0.1uF, Capacitor_SMD:C_0402_1005Metric, symbol Device:C
- added C5: 1uF, Capacitor_SMD:C_0402_1005Metric, symbol Device:C
- added L1: 22uH, Inductor_SMD:L_0402_1005Metric, symbol Device:L
- added U2: XC6206P332MR, Package_TO_SOT_SMD:SOT-23-3, symbol Regulator_Linear:XC6206PxxxMR
- added Y1: 32M, Crystal:Crystal_SMD_3225-4Pin_3.2x2.5mm, symbol Device:Crystal_GND23
Connections:
- net GND: now also J1.2 (Ext), U1.29 (GND), C1.2, C2.2, C3.2, C4.1, C5.1, U2.1 (GND), Y1.2 (G), Y1.3 (G); no longer U1.5 (VDD33/VIO33)
- net at J1.1 (In): now also U1.21 (ANT)
- net at U1.18 (~{X32MO}): now also Y1.1
- net at U1.19 (X32MI): now also Y1.4
- net VCC: now reaches U1.20 (VINTA)
- net VCC: now also U1.5 (VDD33/VIO33), C2.1, C3.1, U2.2 (VO)
- net at U1.22 (VDCIA): now also U1.3 (VDCID), C4.2, C5.2, L1.1
- net at U1.4 (VSW): now also L1.2
- new net +5V: C1.1, U2.3 (VI)
Other:
- moved on the sheet: J1

Commit message: Core
Parts:
- added Y2: 32.768K, Crystal:Crystal_SMD_1210-4Pin_1.2x1.0mm, symbol Device:Crystal_GND23
- C3: value 0.1uF -> 0.47uF
Connections:
- net GND: now also Y2.2 (G), Y2.3 (G)
- net VCC: no longer C3.1, U1.20 (VINTA)
- net X32KI: no longer names the net of U1.1 (PA11)
- net X32KI: now also Y2.1
- net X32KO: no longer names the net of U1.2 (PA10)
- net X32KO: now also Y2.4
- new net: C3.1, U1.20 (VINTA)
Other:
- moved on the sheet: C3
Changed lines of the file:
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@@
-	)
-	(junction
-		(at 44.45 85.09)
-		(diameter 0)
-		(color 0 0 0 0)
 	)
 	(junction
@@
 	(wire
 		(pts
-			(xy 43.18 54.61) (xy 49.53 54.61)
-		)
-		(stroke
-			(width 0)
-			(type default)
-		)
-	)
-	(wire
-		(pts
 			(xy 88.9 78.74) (xy 88.9 73.66)
 		)
@@
 	(wire
 		(pts
-			(xy 44.45 85.09) (xy 49.53 85.09)
-		)
-		(stroke
-			(width 0)
-			(type default)
-		)
-	)
-	(wire
-		(pts
 			(xy 46.99 24.13) (xy 40.64 24.13)
 		)
@@
 	(wire
 		(pts
+			(xy 31.75 57.15) (xy 36.83 57.15)
+		)
+		(stroke
+			(width 0)
+			(type default)
+		)
+	)
+	(wire
+		(pts
 			(xy 34.29 69.85) (xy 34.29 80.01)
 		)
@@
 	(wire
 		(pts
-			(xy 44.45 92.71) (xy 62.23 92.71)
+			(xy 49.53 92.71) (xy 62.23 92.71)
 		)
 		(stroke
@@
 	(wire
 		(pts
+			(xy 36.83 52.07) (xy 36.83 49.53)
+		)
+		(stroke
+			(width 0)
+			(type default)
+		)
+	)
+	(wire
+		(pts
 			(xy 62.23 92.71) (xy 62.23 90.17)
 		)
@@
 	(wire
 		(pts
-			(xy 41.91 85.09) (xy 44.45 85.09)
+			(xy 49.53 52.07) (xy 36.83 52.07)
+		)
+		(stroke
+			(width 0)
+			(type default)
+		)
+	)
+	(wire
+		(pts
+			(xy 36.83 54.61) (xy 49.53 54.61)
 		)
 		(stroke
@@
 	(wire
 		(pts
+			(xy 36.83 49.53) (xy 31.75 49.53)
+		)
+		(stroke
+			(width 0)
+			(type default)
+		)
+	)
+	(wire
+		(pts
 			(xy 33.02 31.75) (xy 46.99 31.75)
 		)
@@
 	(wire
 		(pts
-			(xy 43.18 52.07) (xy 49.53 52.07)
+			(xy 36.83 57.15) (xy 36.83 54.61)
 		)
 		(stroke
@@
 			(width 0)
 			(type default)
-		)
-	)
-	(label "X32KI"
-		(at 43.18 54.61 0)
-		(effects
-			(font
-				(size 1.27 1.27)
-			)
-			(justify left bottom)
-		)
-	)
-	(label "X32KO"
-		(at 43.18 52.07 0)
-		(effects
-			(font
-				(size 1.27 1.27)
-			)
-			(justify left bottom)
 		)
 	)
@@
 	)
 	(symbol
+		(lib_id "Device:Crystal_GND23")
+		(at 31.75 53.34 90)
+		(unit 1)
+		(body_style 1)
+		(exclude_from_sim no)
+		(in_bom yes)
+		(on_board yes)
+		(in_pos_files yes)
+		(dnp no)
+		(fields_autoplaced yes)
+		(property "Reference" "Y2"
+			(at 26.67 52.0699 90)
+			(show_name no)
+			(do_not_autoplace no)
+			(effects
+				(font
+					(size 1.27 1.27)
+				)
+				(justify left)
+			)
+		)
+		(property "Value" "32.768K"
+			(at 26.67 54.6099 90)
+			(show_name no)
+			(do_not_autoplace no)
+			(effects
+				(font
+					(size 1.27 1.27)
+				)
+				(justify left)
+			)
+		)
+		(property "Footprint" "Crystal:Crystal_SMD_1210-4Pin_1.2x1.0mm"
+			(at 31.75 53.34 0)
+			(hide yes)
+			(show_name no)
+			(do_not_autoplace no)
+			(effects
+				(font
+					(size 1.27 1.27)
+				)
+			)
+		)
+		(property "Datasheet" ""
+			(at 31.75 53.34 0)
+			(hide yes)
+			(show_name no)
+			(do_not_autoplace no)
+			(effects
+				(font
+					(size 1.27 1.27)
+				)
+			)
+		)
+		(property "Description" "Four pin crystal, GND on pins 2 and 3"
+			(at 31.75 53.34 0)
+			(hide yes)
+			(show_name no)
+			(do_not_autoplace no)
+			(effects
+				(font
+					(size 1.27 1.27)
+				)
+			)
+		)
+		(property private "KLC_S3.3" "The rectangle is not a symbol body but a graphical element"
+			(at 44.45 53.34 0)
+			(hide yes)
+			(show_name yes)
+			(do_not_autoplace no)
+			(effects
+				(font
+					(size 1.27 1.27)
+				)
+			)
+		)
+		(property private "KLC_S4.1" "Some pins are on 50mil grid to make the symbol small"
+			(at 46.99 53.34 0)
+			(hide yes)
+			(show_name yes)
+			(do_not_autoplace no)
+			(effects
+				(font
+					(size 1.27 1.27)
+				)
+			)
+		)
+		(pin "2"
+		)
+		(pin "4"
+		)
+		(pin "1"
+		)
+		(pin "3"
+		)
+		(instances
+			(project "TinyLamp"
+				(path "/f38cd39d-d88c-4ddb-9850-45d0bcc3e4cb"
+					(reference "Y2")
+					(unit 1)
+				)
+			)
+		)
+	)
+	(symbol
 		(lib_id "Device:C")
 		(at 38.1 69.85 90)
@@
 	)
 	(symbol
-		(lib_id "power:VCC")
-		(at 41.91 85.09 90)
-		(unit 1)
-		(body_style 1)
-		(exclude_from_sim no)
-		(in_bom yes)
-		(on_board yes)
-		(in_pos_files yes)
-		(dnp no)
-		(fields_autoplaced yes)
-		(property "Reference" "#PWR07"
-			(at 45.72 85.09 0)
-			(hide yes)
-			(show_name no)
-			(do_not_autoplace no)
-			(effects
-				(font
-					(size 1.27 1.27)
-				)
-			)
-		)
-		(property "Value" "VCC"
-			(at 38.1 85.0899 90)
-			(show_name no)
-			(do_not_autoplace no)
-			(effects
-				(font
-					(size 1.27 1.27)
-				)
-				(justify left)
-			)
-		)
-		(property "Footprint" ""
-			(at 41.91 85.09 0)
-			(hide yes)
-			(show_name no)
-			(do_not_autoplace no)
-			(effects
-				(font
-					(size 1.27 1.27)
-				)
-			)
-		)
-		(property "Datasheet" ""
-			(at 41.91 85.09 0)
-			(hide yes)
-			(show_name no)
-			(do_not_autoplace no)
-			(effects
-				(font
-					(size 1.27 1.27)
-				)
-			)
-		)
-		(property "Description" "Power symbol creates a global label with name \"VCC\""
-			(at 41.91 85.09 0)
-			(hide yes)
-			(show_name no)
-			(do_not_autoplace no)
-			(effects
-				(font
-					(size 1.27 1.27)
-				)
-			)
-		)
-		(pin "1"
-		)
-		(instances
-			(project "TinyLamp"
-				(path "/f38cd39d-d88c-4ddb-9850-45d0bcc3e4cb"
-					(reference "#PWR07")
-					(unit 1)
-				)
-			)
-		)
-	)
-	(symbol
 		(lib_id "power:+5V")
 		(at 17.78 24.13 0)
@@
 	)
 	(symbol
-		(lib_id "Device:C")
-		(at 44.45 88.9 0)
+		(lib_id "power:GND")
+		(at 36.83 53.34 90)
 		(unit 1)
 		(body_style 1)
@@
 		(dnp no)
 		(fields_autoplaced yes)
+		(property "Reference" "#PWR07"
+			(at 43.18 53.34 0)
+			(hide yes)
+			(show_name no)
+			(do_not_autoplace no)
+			(effects
+				(font
+					(size 1.27 1.27)
+				)
+			)
+		)
+		(property "Value" "GND"
+			(at 40.64 53.3399 90)
+			(show_name no)
+			(do_not_autoplace no)
+			(effects
+				(font
+					(size 1.27 1.27)
+				)
+				(justify right)
+			)
+		)
+		(property "Footprint" ""
+			(at 36.83 53.34 0)
+			(hide yes)
+			(show_name no)
+			(do_not_autoplace no)
+			(effects
+				(font
+					(size 1.27 1.27)
+				)
+			)
+		)
+		(property "Datasheet" ""
+			(at 36.83 53.34 0)
+			(hide yes)
+			(show_name no)
+			(do_not_autoplace no)
+			(effects
+				(font
+					(size 1.27 1.27)
+				)
+			)
+		)
+		(property "Description" "Power symbol creates a global label with name \"GND\" , ground"
+			(at 36.83 53.34 0)
+			(hide yes)
+			(show_name no)
+			(do_not_autoplace no)
+			(effects
+				(font
+					(size 1.27 1.27)
+				)
+			)
+		)
+		(pin "1"
+		)
+		(instances
+			(project "TinyLamp"
+				(path "/f38cd39d-d88c-4ddb-9850-45d0bcc3e4cb"
+					(reference "#PWR07")
+					(unit 1)
+				)
+			)
+		)
+	)
+	(symbol
+		(lib_id "Device:C")
+		(at 49.53 88.9 0)
+		(unit 1)
+		(body_style 1)
+		(exclude_from_sim no)
+		(in_bom yes)
+		(on_board yes)
+		(in_pos_files yes)
+		(dnp no)
 		(property "Reference" "C3"
-			(at 48.26 87.6299 0)
+			(at 44.196 87.122 0)
 			(show_name no)
 			(do_not_autoplace no)
@@
 			)
 		)
-		(property "Value" "0.1uF"
-			(at 48.26 90.1699 0)
+		(property "Value" "0.47uF"
+			(at 40.894 89.408 0)
 			(show_name no)
 			(do_not_autoplace no)
@@
 		)
 		(property "Footprint" "Capacitor_SMD:C_0402_1005Metric"
-			(at 45.4152 92.71 0)
+			(at 50.4952 92.71 0)
 			(hide yes)
 			(show_name no)
@@
 		)
 		(property "Datasheet" ""
-			(at 44.45 88.9 0)
+			(at 49.53 88.9 0)
 			(hide yes)
 			(show_name no)
@@
 		)
 		(property "Description" "Unpolarized capacitor"
-			(at 44.45 88.9 0)
-			(hide yes)
-			(show_name no)
+			(at 49.53 88.9 0)
+			(hide yes)
+			(show_name no)

Commit message: Core
Parts:
- added U3: Opamp_Dual, Package_SO:VSSOP-8_2.3x2mm_P0.5mm, symbol Device:Opamp_Dual
Connections:
- net GND: now also U3.4 (V-)
- net VCC: now also U3.8 (V+)

Commit message: Touch
Parts:
- removed U3: Opamp_Dual, Package_SO:VSSOP-8_2.3x2mm_P0.5mm, symbol Device:Opamp_Dual
Connections:
- net TCH0: now reaches U1.6 (PA8)
- net TCH1: now reaches U1.7 (PA9)
